Commit message: first time working :)

File: teleopvr_description/urdf/teleopvr_gripper_macro.xacro (robot description, xacro)
@@ -2,22 +2,13 @@
 <robot
     xmlns:xacro="http://ros.org/wiki/xacro">
+    <xacro:property name="length" value="0.173" />
+    <xacro:property name="radius1" value="0.020" />
+    <xacro:property name="radius2" value="0.007" />
+    <xacro:property name="hlength" value="0.050" />
     <xacro:macro name="teleopvr_gripper" params="prefix">
         <link name="${prefix}base_link" />
-        <link name="${prefix}tool_tip">
-            <visual>
-                <origin xyz="-0.2 0 0" rpy="0 ${pi/2} 0"/>
-                <geometry>
-                    <mesh filename="package://teleopvr_description/meshes/tool.dae"/>
-                </geometry>
-            </visual>
-            <collision>
-                <origin xyz="-0.2 0 0" rpy="0 ${pi/2} 0"/>
-                <geometry>
-                    <mesh filename="package://teleopvr_description/meshes/tool.dae"/>
-                </geometry>
-            </collision>
-        </link>
+        <link name="${prefix}tool_tip"></link>
         <joint name="${prefix}base_link-${prefix}tool_tip" type="fixed">
-            <origin xyz="0.2 0 0" rpy="0 0 0" />
+            <origin xyz="${length} 0 0" rpy="0 0 0" />
             <parent link="${prefix}base_link" />
             <child link="${prefix}tool_tip" />

File: teleopvr_description/urdf/teleopvr_macro.xacro (robot description, xacro)
@@ -11,5 +11,5 @@
         <xacro:teleopvr_manipulator prefix="${prefix}" />
         <xacro:kinect_camera name="camera" parent="${prefix}robot_base_link">
-            <origin rpy="0 ${pi/2} 0" xyz="0.7 0 1.0" />
+            <origin rpy="${pi} ${pi/2} 0" xyz="0.7 0 1.0" />
         </xacro:kinect_camera>
     </xacro:macro>

Commit message: added gripper stl and updated the moveit collisions

File: teleopvr_description/urdf/teleopvr_gripper_macro.xacro (robot description, xacro)
@@ -7,6 +7,18 @@
     <xacro:property name="hlength" value="0.050" />
     <xacro:macro name="teleopvr_gripper" params="prefix">
-        <link name="${prefix}base_link" />
-        <link name="${prefix}tool_tip"></link>
+        <link name="${prefix}base_link">
+            <visual>
+                <origin rpy="0 ${pi/2} 0" xyz="0 0 0" />
+                <geometry>
+                    <mesh filename="package://teleopvr_description/meshes/tool.dae" />
+                </geometry>
+            </visual>
+            <collision>
+                <geometry>
+                    <mesh filename="package://teleopvr_description/meshes/tool.dae" />
+                </geometry>
+            </collision>
+        </link>
+        <link name="${prefix}tool_tip" />
         <joint name="${prefix}base_link-${prefix}tool_tip" type="fixed">
             <origin xyz="${length} 0 0" rpy="0 0 0" />

Commit message: all calibration nodes are done

File: teleopvr_description/urdf/teleopvr_gripper_macro.xacro (robot description, xacro)
@@ -22,5 +22,5 @@
         <link name="${prefix}tool_tip" />
         <joint name="${prefix}base_link-${prefix}tool_tip" type="fixed">
-            <origin xyz="${length} 0 0" rpy="0 0 0" />
+            <origin xyz="${length} 0 0" rpy="0 ${pi/2} 0" />
             <parent link="${prefix}base_link" />
             <child link="${prefix}tool_tip" />

File: teleopvr_description/urdf/teleopvr_macro.xacro (robot description, xacro)
@@ -11,5 +11,7 @@
         <xacro:teleopvr_manipulator prefix="${prefix}" />
         <xacro:kinect_camera name="camera" parent="${prefix}robot_base_link">
-            <origin rpy="${pi} ${pi/2} 0" xyz="0.7 0 1.0" />
+            <origin
+                xyz="0.72840281694 -0.249040209926 1.0"
+                rpy="${pi} ${pi/2} 0" />
         </xacro:kinect_camera>
     </xacro:macro>
