Commit message: created new package with gripper for better organization

File: teleopvr_description/urdf/teleopvr_manipulator_macro.xacro (robot description, xacro)
@@ -6,5 +6,5 @@
     <xacro:include filename="$(find fanuc_lrmate200id_support)/urdf/lrmate200id_macro.xacro"/>
     <!-- include end effector gripper -->
-    <xacro:include filename="$(find teleopvr_description)/urdf/teleopvr_gripper_macro.xacro"/>
+    <xacro:include filename="$(find teleopvr_gripper_description)/urdf/teleopvr_gripper_macro.xacro"/>
     <!-- manipulator macro -->
     <xacro:macro name="teleopvr_manipulator" params="prefix">

File: teleopvr_gripper_description/urdf/teleopvr_gripper_macro.xacro (robot description, xacro)
@@ -11,10 +11,10 @@
                 <origin rpy="0 ${pi/2} 0" xyz="0 0 0" />
                 <geometry>
-                    <mesh filename="package://teleopvr_description/meshes/tool.dae" />
+                    <mesh filename="package://teleopvr_gripper_description/meshes/tool.dae" />
                 </geometry>
             </visual>
             <collision>
                 <geometry>
-                    <mesh filename="package://teleopvr_description/meshes/tool.dae" />
+                    <mesh filename="package://teleopvr_gripper_description/meshes/tool.dae" />
                 </geometry>
             </collision>
