Commit message: updated robot configuration for new robot

File: teleopvr_description/urdf/teleopvr_macro.xacro (robot description, xacro)
@@ -1,18 +1,9 @@
 <?xml version="1.0" ?>
-<robot
-    xmlns:xacro="http://ros.org/wiki/xacro">
+<robot xmlns:xacro="http://ros.org/wiki/xacro">
     <!-- include the manipulator xacro -->
     <xacro:include filename="$(find teleopvr_description)/urdf/teleopvr_manipulator_macro.xacro"/>
-    <!-- include the kinetic xacro -->
-    <xacro:include filename="$(find hector_xacro_tools)/urdf/inertia_tensors.urdf.xacro"/>
-    <xacro:include filename="$(find hector_sensors_description)/urdf/kinect_camera.urdf.xacro" />
     <!-- macro defining the whole robot -->
     <xacro:macro name="teleopvr" params="prefix">
         <xacro:teleopvr_manipulator prefix="${prefix}" />
-        <xacro:kinect_camera name="camera" parent="${prefix}robot_base_link">
-            <origin
-                xyz="0.68335329 -0.1191058 1.03896683"
-                rpy="3.0303556  1.7643787 -0.0945628" />
-        </xacro:kinect_camera>
     </xacro:macro>
 </robot>

File: teleopvr_description/urdf/teleopvr_manipulator_macro.xacro (robot description, xacro)
@@ -1,8 +1,7 @@
 <?xml version="1.0"?>
-<robot
-    xmlns:xacro="http://ros.org/wiki/xacro">
+<robot xmlns:xacro="http://ros.org/wiki/xacro">
     <!-- xacro includes -->
     <!-- include lrmate200id robot -->
-    <xacro:include filename="$(find fanuc_lrmate200id_support)/urdf/lrmate200id_macro.xacro"/>
+    <xacro:include filename="$(find fanuc_m16ib_support)/urdf/m16ib20_macro.xacro"/>
     <!-- include end effector gripper -->
     <xacro:include filename="$(find teleopvr_gripper_description)/urdf/teleopvr_gripper_macro.xacro"/>
@@ -10,5 +9,5 @@
     <xacro:macro name="teleopvr_manipulator" params="prefix">
         <!-- lrmate200id robot -->
-        <xacro:fanuc_lrmate200id prefix="${prefix}robot_" />
+        <xacro:fanuc_m16ib20 prefix="${prefix}robot_" />
         <!-- end effector gripper -->
         <xacro:teleopvr_gripper prefix="${prefix}eef_" />
